File: KiCAD/LED_pixel_board/LED_pixel_board.kicad_sch (KiCad schematic)
At the start: 60 parts, among them J3 Screw_Terminal_01x02, Y1 ASCO

Commit message: added a lot of captures + some schematic updates
Parts:
- added J1: S1, symbol Connector_Generic:Conn_02x02_Counter_Clockwise
Connections:
- net GND2: now also J1.2 (Pin_2)
- net at TP9.1, U6.48: now also J1.1 (Pin_1)
- no-connect marks 3 -> 5
Changed lines of the file:
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@@
 	)
 	(junction
+		(at 153.67 43.18)
+		(diameter 0)
+		(color 0 0 0 0)
+	)
+	(junction
 		(at 78.74 146.05)
 		(diameter 0)
@@
 	)
 	(no_connect
+		(at 181.61 26.67)
+	)
+	(no_connect
+		(at 181.61 29.21)
+	)
+	(no_connect
 		(at 205.74 46.99)
 	)
@@
 	(wire
 		(pts
+			(xy 153.67 43.18) (xy 166.37 43.18)
+		)
+		(stroke
+			(width 0)
+			(type default)
+		)
+	)
+	(wire
+		(pts
 			(xy 203.2 195.58) (xy 203.2 203.2)
 		)
@@
 	(wire
 		(pts
-			(xy 120.65 43.18) (xy 166.37 43.18)
+			(xy 120.65 43.18) (xy 153.67 43.18)
 		)
 		(stroke
@@
 	(wire
 		(pts
+			(xy 165.1 29.21) (xy 168.91 29.21)
+		)
+		(stroke
+			(width 0)
+			(type default)
+		)
+	)
+	(wire
+		(pts
 			(xy 205.74 25.4) (xy 205.74 22.86)
 		)
@@
 	(wire
 		(pts
+			(xy 165.1 31.75) (xy 165.1 29.21)
+		)
+		(stroke
+			(width 0)
+			(type default)
+		)
+	)
+	(wire
+		(pts
 			(xy 135.89 199.39) (xy 135.89 153.67)
 		)
@@
 	(wire
 		(pts
+			(xy 153.67 26.67) (xy 168.91 26.67)
+		)
+		(stroke
+			(width 0)
+			(type default)
+		)
+	)
+	(wire
+		(pts
 			(xy 73.66 27.94) (xy 69.85 27.94)
 		)
@@
 	(wire
 		(pts
+			(xy 153.67 43.18) (xy 153.67 26.67)
+		)
+		(stroke
+			(width 0)
+			(type default)
+		)
+	)
+	(wire
+		(pts
 			(xy 69.85 20.32) (xy 69.85 17.78)
 		)
@@
 	)
 	(symbol
+		(lib_id "power:GND2")
+		(at 165.1 31.75 0)
+		(unit 1)
+		(exclude_from_sim no)
+		(in_bom yes)
+		(on_board yes)
+		(dnp no)
+		(fields_autoplaced yes)
+		(property "Reference" "#PWR080"
+			(at 165.1 38.1 0)
+			(effects
+				(font
+					(size 1.27 1.27)
+				)
+				(hide yes)
+			)
+		)
+		(property "Value" "GND2"
+			(at 165.1 36.83 0)
+			(effects
+				(font
+					(size 1.27 1.27)
+				)
+			)
+		)
+		(property "Footprint" ""
+			(at 165.1 31.75 0)
+			(effects
+				(font
+					(size 1.27 1.27)
+				)
+				(hide yes)
+			)
+		)
+		(property "Datasheet" ""
+			(at 165.1 31.75 0)
+			(effects
+				(font
+					(size 1.27 1.27)
+				)
+				(hide yes)
+			)
+		)
+		(property "Description" "Power symbol creates a global label with name \"GND2\" , ground"
+			(at 165.1 31.75 0)
+			(effects
+				(font
+					(size 1.27 1.27)
+				)
+				(hide yes)
+			)
+		)
+		(pin "1"
+		)
+		(instances
+			(project "LED_pixel_board"
+				(path "/64f17c8a-724c-4bac-a14e-8a622f982c2e"
+					(reference "#PWR080")
+					(unit 1)
+				)
+			)
+		)
+	)
+	(symbol
 		(lib_id "Device:C")
 		(at 184.15 59.69 0)
@@
 					(unit 1)
 				)
+			)
+		)
+	)
+	(symbol
+		(lib_id "Connector_Generic:Conn_02x02_Counter_Clockwise")
+		(at 173.99 26.67 0)
+		(unit 1)
+		(exclude_from_sim no)
+		(in_bom yes)
+		(on_board yes)
+		(dnp no)
+		(fields_autoplaced yes)
+		(property "Reference" "J1"
+			(at 175.26 20.32 0)
+			(effects
+				(font
+					(size 1.27 1.27)
+				)
+			)
+		)
+		(property "Value" "S1"
+			(at 175.26 22.86 0)
+			(effects
+				(font
+					(size 1.27 1.27)
+				)
+			)
+		)
+		(property "Footprint" ""
+			(at 173.99 26.67 0)
+			(effects
+				(font
+					(size 1.27 1.27)
+				)
+				(hide yes)
+			)
+		)
+		(property "Datasheet" "~"
+			(at 173.99 26.67 0)
+			(effects
+				(font
+					(size 1.27 1.27)
+				)
+				(hide yes)
+			)
+		)
+		(property "Description" "Generic connector, double row, 02x02, counter clockwise pin numbering scheme (similar to DIP package numbering), script generated (kicad-library-utils/schlib/autogen/connector/)"
+			(at 173.99 26.67 0)
+			(effects
+				(font
+					(size 1.27 1.27)
+				)
+				(hide yes)
+			)
+		)
+		(pin "1"
+		)
+		(pin "2"
+		)
+		(pin "4"
+		)
+		(pin "3"
+		)
+		(instances
+			(project ""
+				(path "/64f17c8a-724c-4bac-a14e-8a622f982c2e"
+					(reference "J1")
+					(unit 1)
+				)
